File: accel-breakout.sch (KiCad schematic (older format))
At the start: 14 parts

Commit message: sch done
Parts:
- removed J?: Conn_01x08, symbol Connector_Generic:Conn_01x08
- added C3: 10u, symbol Device:C
- added C6: 100n, symbol Device:C
- added J?: Conn_01x09, symbol Connector_Generic:Conn_01x09
- added U2: LIS302DL, symbol accel-gyro:LIS302DL
- gave numbers to parts that had none: 13
Connections:
- wire segments 60 -> 99
Other:
- note added: "L3GD20\nX: 1->12\nY: 4->1\nZ: up"
- note added: "LIS302DL\nX: 1->6\nY: 8->6\nZ: up"

Commit message: pcb done
Parts:
- removed C3: 10u, symbol Device:C
- added C3: 10u, Capacitor_SMD:C_0805_2012Metric, symbol Device:CP
- C1: value CP -> 10u; footprint (none) -> Capacitor_SMD:C_0805_2012Metric
- C2, C4, C5, C6: footprint (none) -> Capacitor_SMD:C_0805_2012Metric
- J1: renamed from J?; footprint (none) -> Connector_PinHeader_2.54mm:PinHeader_1x09_P2.54mm_Vertical
- JP1, JP2, JP3, JP4: footprint (none) -> Jumper:SolderJumper-2_P1.3mm_Open_RoundedPad1.0x1.5mm
- R1, R2, R3, R4: footprint (none) -> Resistor_SMD:R_0805_2012Metric
- U1: footprint LGA-16 -> accel-gyro:LGA-16
- U2: footprint (none) -> accel-gyro:LIS302DL
Changed lines of the file:
@@
 F 0 "U1" H 5100 1314 50  0000 C CNN
 F 1 "L3GD20" H 5100 1223 50  0000 C CNN
-F 2 "LGA-16" H 5100 2000 50  0001 C CIN
+F 2 "accel-gyro:LGA-16" H 5100 2000 50  0001 C CIN
 F 3 "http://www.st.com/st-web-ui/static/active/en/resource/technical/document/datasheet/DM00036465.pdf" H 5100 2000 50  0001 C CNN
 	1    5100 2000
@@
 F 0 "R1" H 6120 1096 50  0000 L CNN
 F 1 "10k" H 6120 1005 50  0000 L CNN
-F 2 "" V 5980 1050 50  0001 C CNN
+F 2 "Resistor_SMD:R_0805_2012Metric" V 5980 1050 50  0001 C CNN
 F 3 "~" H 6050 1050 50  0001 C CNN
 	1    6050 1050
@@
 F 0 "R2" H 6370 1096 50  0000 L CNN
 F 1 "10k" H 6370 1005 50  0000 L CNN
-F 2 "" V 6230 1050 50  0001 C CNN
+F 2 "Resistor_SMD:R_0805_2012Metric" V 6230 1050 50  0001 C CNN
 F 3 "~" H 6300 1050 50  0001 C CNN
 	1    6300 1050
@@
 F 0 "JP1" V 6050 1518 50  0000 L CNN
 F 1 "SolderJumper_2_Open" V 6095 1518 50  0001 L CNN
-F 2 "" H 6050 1450 50  0001 C CNN
+F 2 "Jumper:SolderJumper-2_P1.3mm_Open_RoundedPad1.0x1.5mm" H 6050 1450 50  0001 C CNN
 F 3 "~" H 6050 1450 50  0001 C CNN
 	1    6050 1450
@@
 F 0 "JP2" V 6300 1518 50  0000 L CNN
 F 1 "SolderJumper_2_Open" V 6345 1518 50  0001 L CNN
-F 2 "" H 6300 1450 50  0001 C CNN
+F 2 "Jumper:SolderJumper-2_P1.3mm_Open_RoundedPad1.0x1.5mm" H 6300 1450 50  0001 C CNN
 F 3 "~" H 6300 1450 50  0001 C CNN
 	1    6300 1450
@@
 F 0 "R3" H 6620 1096 50  0000 L CNN
 F 1 "10k" H 6620 1005 50  0000 L CNN
-F 2 "" V 6480 1050 50  0001 C CNN
+F 2 "Resistor_SMD:R_0805_2012Metric" V 6480 1050 50  0001 C CNN
 F 3 "~" H 6550 1050 50  0001 C CNN
 	1    6550 1050
@@
 F 0 "R4" H 6870 1096 50  0000 L CNN
 F 1 "10k" H 6870 1005 50  0000 L CNN
-F 2 "" V 6730 1050 50  0001 C CNN
+F 2 "Resistor_SMD:R_0805_2012Metric" V 6730 1050 50  0001 C CNN
 F 3 "~" H 6800 1050 50  0001 C CNN
 	1    6800 1050
@@
 F 0 "JP3" V 6550 1518 50  0000 L CNN
 F 1 "SolderJumper_2_Open" V 6595 1518 50  0001 L CNN
-F 2 "" H 6550 1450 50  0001 C CNN
+F 2 "Jumper:SolderJumper-2_P1.3mm_Open_RoundedPad1.0x1.5mm" H 6550 1450 50  0001 C CNN
 F 3 "~" H 6550 1450 50  0001 C CNN
 	1    6550 1450
@@
 F 0 "JP4" V 6800 1518 50  0000 L CNN
 F 1 "SolderJumper_2_Open" V 6845 1518 50  0001 L CNN
-F 2 "" H 6800 1450 50  0001 C CNN
+F 2 "Jumper:SolderJumper-2_P1.3mm_Open_RoundedPad1.0x1.5mm" H 6800 1450 50  0001 C CNN
 F 3 "~" H 6800 1450 50  0001 C CNN
 	1    6800 1450
@@
 F 0 "C4" H 4065 1546 50  0000 L CNN
 F 1 "0.1u" H 4065 1455 50  0000 L CNN
-F 2 "" H 3988 1350 50  0001 C CNN
+F 2 "Capacitor_SMD:C_0805_2012Metric" H 3988 1350 50  0001 C CNN
 F 3 "~" H 3950 1500 50  0001 C CNN
 	1    3950 1500
@@
 F 0 "C2" H 3615 1546 50  0000 L CNN
 F 1 "0.1u" H 3615 1455 50  0000 L CNN
-F 2 "" H 3538 1350 50  0001 C CNN
+F 2 "Capacitor_SMD:C_0805_2012Metric" H 3538 1350 50  0001 C CNN
 F 3 "~" H 3500 1500 50  0001 C CNN
 	1    3500 1500
@@
 P 3150 1500
 F 0 "C1" H 3268 1546 50  0000 L CNN
-F 1 "CP" H 3268 1455 50  0000 L CNN
-F 2 "" H 3188 1350 50  0001 C CNN
+F 1 "10u" H 3268 1455 50  0000 L CNN
+F 2 "Capacitor_SMD:C_0805_2012Metric" H 3188 1350 50  0001 C CNN
 F 3 "~" H 3150 1500 50  0001 C CNN
 	1    3150 1500
@@
 F 0 "C5" H 4065 1996 50  0000 L CNN
 F 1 "1n" H 4065 1905 50  0000 L CNN
-F 2 "" H 3988 1800 50  0001 C CNN
+F 2 "Capacitor_SMD:C_0805_2012Metric" H 3988 1800 50  0001 C CNN
 F 3 "~" H 3950 1950 50  0001 C CNN
 F 4 "16V" H 3950 1950 50  0001 C CNN "Voltage"
@@
 F 0 "C6" H 4315 3446 50  0000 L CNN
 F 1 "100n" H 4315 3355 50  0000 L CNN
-F 2 "" H 4238 3250 50  0001 C CNN
+F 2 "Capacitor_SMD:C_0805_2012Metric" H 4238 3250 50  0001 C CNN
 F 3 "~" H 4200 3400 50  0001 C CNN
 	1    4200 3400
-	1    0    0    -1
-$EndComp
-$Comp
-L Device:C C3
-U 1 1 5AC63053
-P 3850 3400
-F 0 "C3" H 3965 3446 50  0000 L CNN
-F 1 "10u" H 3965 3355 50  0000 L CNN
-F 2 "" H 3888 3250 50  0001 C CNN
-F 3 "~" H 3850 3400 50  0001 C CNN
-	1    3850 3400
 	1    0    0    -1
 $EndComp
@@
 F 0 "U2" H 5150 4075 50  0000 C CNN
 F 1 "LIS302DL" H 5150 3984 50  0000 C CNN
-F 2 "" H 5350 3700 50  0001 C CNN
+F 2 "accel-gyro:LIS302DL" H 5350 3700 50  0001 C CNN
 F 3 "" H 5350 3700 50  0001 C CNN
 	1    5150 3500
@@
 	6800 1600 6800 2300
 $Comp
-L Connector_Generic:Conn_01x09 J?
+L Connector_Generic:Conn_01x09 J1
 U 1 1 5AC794B2
 P 7300 2100
-F 0 "J?" H 7380 2142 50  0000 L CNN
+F 0 "J1" H 7380 2142 50  0000 L CNN
 F 1 "Conn_01x09" H 7380 2051 50  0000 L CNN
-F 2 "" H 7300 2100 50  0001 C CNN
+F 2 "Connector_PinHeader_2.54mm:PinHeader_1x09_P2.54mm_Vertical" H 7300 2100 50  0001 C CNN
 F 3 "~" H 7300 2100 50  0001 C CNN
 	1    7300 2100
@@
 Wire Wire Line
 	7050 2500 7050 2700
+$Comp
+L Device:CP C3
+U 1 1 5AC8883C
+P 3850 3400
+F 0 "C3" H 3968 3446 50  0000 L CNN
+F 1 "10u" H 3968 3355 50  0000 L CNN
+F 2 "Capacitor_SMD:C_0805_2012Metric" H 3888 3250 50  0001 C CNN
+F 3 "~" H 3850 3400 50  0001 C CNN
+	1    3850 3400
+	1    0    0    -1
+$EndComp
 $EndSCHEMATC
