File: accel-breakout.kicad_pcb (KiCad board)
At the start: 2 copper layers, 26 x 24 mm, 19 parts, among them J1 Conn_01x09, M1 TestPoint_Plated_Hole_D2.0mm, M2 TestPoint_Plated_Hole_D2.0mm, U1 L3GD20, U2 LIS302DL

Commit message: pcb: added b.silk
Other:
- board text added: "3V3"
- board text added: "CS L3GD20"
- board text added: "CS LIS302DL"
- board text added: "GND"
- board text added: "INT1"
- board text added: "INT2"
- board text added: "SCL/SPC"
- board text added: "SDA/SDI"
- board text added: "SDO"
- board text added: "github.com/ dimka-rs/ accel-breakout"
Changed lines of the file:
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@@
   (general
     (thickness 1.6)
-    (drawings 4)
+    (drawings 14)
     (tracks 266)
     (zones 0)
@@
   (page A4)
   (layers
-    (0 F.Cu signal)
+    (0 F.Cu signal hide)
     (31 B.Cu signal)
     (32 B.Adhes user)
@@
     (visible_elements FFFDFFFF)
     (pcbplotparams
-      (layerselection 0x010fc_ffffffff)
-      (usegerberextensions false)
+      (layerselection 0x010f0_ffffffff)
+      (usegerberextensions true)
       (usegerberattributes false)
       (usegerberadvancedattributes false)
@@
       (outputformat 1)
       (mirror false)
-      (drillshape 1)
+      (drillshape 0)
       (scaleselection 1)
-      (outputdirectory ""))
+      (outputdirectory gerbers))
   )
   (net 0 "")
@@
     (pad 1 thru_hole circle (at 0 0) (size 3 3) (drill 2) (layers *.Cu *.Mask))
   )
+  (gr_text 3V3 (at 132.8 101.1) (layer B.SilkS)
+    (effects (font (size 1.5 1.5) (thickness 0.3)) (justify mirror))
+  )
+  (gr_text GND (at 132.8 98.6) (layer B.SilkS)
+    (effects (font (size 1.5 1.5) (thickness 0.3)) (justify mirror))
+  )
+  (gr_text INT2 (at 133 96.1) (layer B.SilkS)
+    (effects (font (size 1.5 1.5) (thickness 0.3)) (justify mirror))
+  )
+  (gr_text INT1 (at 133 93.5) (layer B.SilkS)
+    (effects (font (size 1.5 1.5) (thickness 0.3)) (justify mirror))
+  )
+  (gr_text "CS LIS302DL" (at 137.9 90.8) (layer B.SilkS)
+    (effects (font (size 1.5 1.5) (thickness 0.3)) (justify mirror))
+  )
+  (gr_text "CS L3GD20" (at 137.1 88.4) (layer B.SilkS)
+    (effects (font (size 1.5 1.5) (thickness 0.3)) (justify mirror))
+  )
+  (gr_text SDO (at 133 85.8) (layer B.SilkS)
+    (effects (font (size 1.5 1.5) (thickness 0.3)) (justify mirror))
+  )
+  (gr_text SDA/SDI (at 135.6 83.3) (layer B.SilkS)
+    (effects (font (size 1.5 1.5) (thickness 0.3)) (justify mirror))
+  )
+  (gr_text SCL/SPC (at 135.9 80.8) (layer B.SilkS)
+    (effects (font (size 1.5 1.5) (thickness 0.3)) (justify mirror))
+  )
+  (gr_text "github.com/\ndimka-rs/\naccel-breakout" (at 148.6 91 270) (layer B.SilkS)
+    (effects (font (size 1.5 1.5) (thickness 0.3)) (justify mirror))
+  )
   (gr_line (start 153 79) (end 127 79) (layer Edge.Cuts) (width 0.15))
